File: Quadrifilar_antenna/Quadrifilar_antenna_A/Quadrifilar_antenna.kicad_pcb (KiCad board)
At the start: 2 copper layers, 95 x 95 mm, 8 parts

Commit message: Minor update to part A
Parts:
- added N1: FeedNetwork (Part B), Quadrifilar_antenna:partB, F.Cu at (197.2, 135.3)
- added N2: Balun (Part C), Quadrifilar_antenna:partC, F.Cu at (198.7, 135.3)
